File: DayNight/Setup/LightSensorWiring.sch (EAGLE design)
At the start: 11 parts, among them Q1 2N3904

Commit message: Eeprom: ^5 update
Parts:
- R2: value 500 -> 10k
Changed lines of the file:
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@@
 <part name="U$1" library="Documentation" deviceset="IRRIGATE7" device=""/>
 <part name="Q1" library="Q-NPN" deviceset="NPN" device="SOT23" value="2N3904"/>
-<part name="R2" library="R-C" deviceset="R" device="0805" value="500"/>
+<part name="R2" library="R-C" deviceset="R" device="0805" value="10k"/>
 <part name="R3" library="R-C" deviceset="R" device="0805" value="100k"/>
 <part name="R4" library="R-C" deviceset="R" device="0805" value="10k"/>
