File: KNL/Setup/KNLWiring.sch (EAGLE design)
At the start: 31 parts

Commit message: i2c-debug: for ^5
Parts:
- removed D3: RD, D-LED:LED5MM
- added R2: 10k, R-C:R0805
Connections:
- net N$2: now also R2.2; no longer D3.A, R1.1
- net N$22: now also R2.1; no longer D3.K
- net N$34: now also R1.1
Other:
- note added: "CAT5 CABLE 1"
- note added: "CAT5 CABLE 2"
- note added: "SOLAR PANEL AS LIGHT SENSOR ADC0 = SLP003*1/11"
- note removed: "LIGHT SENSOR"
- moved on the sheet: D1, D2, R1
